File: KicadJE_3340_Experiment/KicadJE_3340_Experiment.sch (KiCad schematic (older format))
At the start: 0 parts

Commit message: two sub sheets made ready
incomplete
Changed lines of the file:
@@
 $Descr A4 11693 8268
 encoding utf-8
-Sheet 1 2
+Sheet 1 3
 Title ""
 Date ""
@@
 F1 "KicadJE_AS3340_datasheet.sch" 50
 $EndSheet
+$Sheet
+S 3000 5000 2000 2500
+U 5E62ACA1
+F0 "KicadJE_AS3340_prophet8" 50
+F1 "KicadJE_AS3340_prophet8.sch" 50
+$EndSheet
 $EndSCHEMATC

Commit message: AS 3340 JE initiated
Changed lines of the file:
@@
 $Descr A4 11693 8268
 encoding utf-8
-Sheet 1 3
+Sheet 1 4
 Title ""
 Date "2020-02-29"
@@
 $EndDescr
 $Sheet
-S 750  5000 1750 2500
+S 725  800  1750 2500
 U 5E4B0DD9
 F0 "KicadJE_AS3340_datasheet.sch" 50
@@
 $EndSheet
 $Sheet
-S 3000 5000 2000 2500
+S 2975 800  2000 2500
 U 5E62ACA1
 F0 "KicadJE_AS3340_prophet8" 50
 F1 "KicadJE_AS3340_prophet8.sch" 50
 $EndSheet
+$Sheet
+S 5450 800  2050 2475
+U 5F49A670
+F0 "JE_AC3340_RevA" 34
+F1 "JE_AC3340_RevA.sch" 34
+$EndSheet
 $EndSCHEMATC
