File: KicadJE_3340_Experiment/KicadJE_AS3340_prophet8.sch (KiCad schematic (older format))
At the start: 53 parts, among them J301 ADSRGate, J302 ADSR, P301 Doepfer_Power_10pin, Q302 MMBT3904, Q303 MMBT3904, Q304 MMBT3904, U301 TL072

Commit message: protection initiated
prophet circuit initiated
Parts:
- removed C305: 10n, Capacitor_SMD:C_0805_2012Metric_Pad1.15x1.40mm_HandSolder, symbol Device:C
- removed U?: TLC555, AJ-Dropbox-Kicad:AJ_SO-8_5.3x6.2mm_P1.27mm, symbol Timer:TLC555
- added C? (x2): 1u, Capacitor_SMD:C_1206_3216Metric_Pad1.42x1.75mm_HandSolder, symbol Device:C
- added C? (x3): 100n, Capacitor_SMD:C_0805_2012Metric_Pad1.15x1.40mm_HandSolder, symbol Device:C
- added C? (x4): 1n, Capacitor_SMD:C_0805_2012Metric_Pad1.15x1.40mm_HandSolder, symbol Device:C
- added C? (x2): 10n, Capacitor_SMD:C_0805_2012Metric_Pad1.15x1.40mm_HandSolder, symbol Device:C
- added D?: LED, LED_SMD:LED_0805_2012Metric_Pad1.15x1.40mm_HandSolder, symbol Device:LED
- added D?: 1N4148, Diode_SMD:D_SOD-123, symbol Device:D
- added D? (x2): 1N1007, Diode_SMD:D_SOD-123, symbol Device:D
- added J?: In1.1, AJ-Dropbox-Kicad:PJ301SM, symbol Connector:AudioJack2_SwitchT
- added J?: In1.2, AJ-Dropbox-Kicad:PJ301SM, symbol Connector:AudioJack2_SwitchT
- added J?: RampOut1, AJ-Dropbox-Kicad:PJ301SM, symbol Connector:AudioJack2_SwitchT
- added J?: SS_In2, AJ-Dropbox-Kicad:PJ301SM, symbol Connector:AudioJack2_SwitchT
- added J?: PulseOut2, AJ-Dropbox-Kicad:PJ301SM, symbol Connector:AudioJack2_SwitchT
- added J?: In1.3, AJ-Dropbox-Kicad:PJ301SM, symbol Connector:AudioJack2_SwitchT
- added J?: SawOut3, AJ-Dropbox-Kicad:PJ301SM, symbol Connector:AudioJack2_SwitchT
- added J?: HS_In3, AJ-Dropbox-Kicad:PJ301SM, symbol Connector:AudioJack2_SwitchT
- added J?: FM_In4, AJ-Dropbox-Kicad:PJ301SM, symbol Connector:AudioJack2_SwitchT
- added J?: PWM_In5, AJ-Dropbox-Kicad:PJ301SM, symbol Connector:AudioJack2_SwitchT
- added P?: HEADER_2x5_Doepfer, Connector_IDC:IDC-Header_2x05_P2.54mm_Vertical, symbol Eurorack:HEADER_2x5_Doepfer
- added R? (x2): 20k, Resistor_SMD:R_0805_2012Metric_Pad1.15x1.40mm_HandSolder, symbol Device:R
- added R? (x3): 100k, Resistor_SMD:R_0805_2012Metric_Pad1.15x1.40mm_HandSolder, symbol Device:R
- added R? (x4): 47k, Resistor_SMD:R_0805_2012Metric_Pad1.15x1.40mm_HandSolder, symbol Device:R
- added R? (x3): 1k, Resistor_SMD:R_0805_2012Metric_Pad1.15x1.40mm_HandSolder, symbol Device:R
- added R? (x5): 470R, Resistor_SMD:R_0805_2012Metric_Pad1.15x1.40mm_HandSolder, symbol Device:R
- added R?: 22k, Resistor_SMD:R_0805_2012Metric_Pad1.15x1.40mm_HandSolder, symbol Device:R
- added R? (x2): 1M, Resistor_SMD:R_0805_2012Metric_Pad1.15x1.40mm_HandSolder, symbol Device:R
- added R?: 1k8, Resistor_SMD:R_0805_2012Metric_Pad1.15x1.40mm_HandSolder, symbol Device:R
- added R?: 100R, Resistor_SMD:R_0805_2012Metric_Pad1.15x1.40mm_HandSolder, symbol Device:R
- added R?: Open, Resistor_SMD:R_0805_2012Metric_Pad1.15x1.40mm_HandSolder, symbol Device:R
- added R?: 0R, Resistor_SMD:R_0805_2012Metric_Pad1.15x1.40mm_HandSolder, symbol Device:R
- added R?: 360k, Resistor_SMD:R_0805_2012Metric_Pad1.15x1.40mm_HandSolder, symbol Device:R
- added R?: 5k6, Resistor_SMD:R_0805_2012Metric_Pad1.15x1.40mm_HandSolder, symbol Device:R
- added R?: 24k, Resistor_SMD:R_0805_2012Metric_Pad1.15x1.40mm_HandSolder, symbol Device:R
- added R?: 680R, Resistor_SMD:R_0805_2012Metric_Pad1.15x1.40mm_HandSolder, symbol Device:R
- added R?: 1M5, Resistor_SMD:R_0805_2012Metric_Pad1.15x1.40mm_HandSolder, symbol Device:R
- added RV?: 1M Release, AJ-Dropbox-Kicad:Potentiometer_China_RK09_Single_Vertical_AJ, symbol Envelope-cache-2018-08-04-13-00-04:POT
- added RV?: 20K HF Track, AJ-Dropbox-Kicad:Potentiometer_China_RK09_Single_Vertical_AJ, symbol Envelope-cache-2018-08-04-13-00-04:POT
- added RV?: 10k, symbol Device:R_POT_TRIM
- added SW? (x2): Inv/NonInv, AJ-Dropbox-Kicad:SP1MS1, symbol Switch:SW_SPDT
- added U?: TL082, AJ-Dropbox-Kicad:AJ_SO-8_5.3x6.2mm_P1.27mm, symbol Amplifier_Operational:TL082
- added U? (x2): TL082, symbol Amplifier_Operational:TL082
- added U?: AS3340, symbol Audio:AS3340
Connections:
- net labels added: +12L, -12VA, CVIn1, FM_Lin_In4, HardSyncIn3, In1, In2, Inv1, Inv2, Out1, Out2, PWM_In5, SoftSyncIn2, VP_2, VSO_3, VTO_1, Vee
- wire segments 167 -> 359
Other:
- moved on the sheet: C?, D?, J?, P?, Q?, R?, RV?, SW?, SW?A, SW?B, U?A, U?B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

Commit message: -5V
Parts:
- removed P301: Doepfer_Power_10pin, Connectors_IDC:IDC-Header_2x05_Pitch2.54mm_Straight, symbol Eurorack:Doepfer_Power_10pin
- removed R?: 680R, Resistor_SMD:R_0805_2012Metric_Pad1.15x1.40mm_HandSolder, symbol Device:R
- removed U?: TL082, AJ-Dropbox-Kicad:AJ_SO-8_5.3x6.2mm_P1.27mm, symbol Amplifier_Operational:TL082
- removed U? (x2): TL082, symbol Amplifier_Operational:TL082
- added U? (x3): TL072, AJ-Dropbox-Kicad:AJ_SO-8_5.3x6.2mm_P1.27mm, symbol Amplifier_Operational:TL072
- added U?: L79L05_SOT89, Package_TO_SOT_SMD:SOT-89-3, symbol Regulator_Linear:L79L05_SOT89
Connections:
- net +12L: now also U301.8 (V+), U?.8 (V+)
- net +12V: no longer U301.8 (V+)
- net -12V: no longer C304.2, U301.4 (V-)
- net -12VA: now also U301.4 (V-), U?.2 (VI), U?.4 (V-)
- net GND: now also U?.1 (GND)
- net Inv1: now also U?.2 (-)
- net Inv2: now also U?.6 (-)
- net Out1: now also U?.1
- net Out2: now also U?.7
- net at R?.2, SW?.3 (C): now also U?.3 (+)
- net at R?.2, SW?.3 (C): now also U?.5 (+)
- new net -5V: C304.2, U?.3 (VO)
Other:
- moved on the sheet: C?, D?, J?, P?, Q?, R?, RV?, SW?, SW?A, SW?B, U?A, U?B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

Commit message: T8 coming alive
Parts:
- removed C301, C303: 1u, Capacitor_SMD:C_1206_3216Metric_Pad1.42x1.75mm_HandSolder, symbol Device:C
- removed D301, D302: 1N1007, Diode_SMD:D_SOD-123, symbol Device:D
- removed J?: In1.3, AJ-Dropbox-Kicad:PJ301SM, symbol Connector:AudioJack2_SwitchT
- removed R?: 100k, Resistor_SMD:R_0805_2012Metric_Pad1.15x1.40mm_HandSolder, symbol Device:R
- removed R?: 1M, Resistor_SMD:R_0805_2012Metric_Pad1.15x1.40mm_HandSolder, symbol Device:R
- removed RV?: 20K HF Track, AJ-Dropbox-Kicad:Potentiometer_China_RK09_Single_Vertical_AJ, symbol Envelope-cache-2018-08-04-13-00-04:POT
- added C?: 100n, Capacitor_SMD:C_0805_2012Metric_Pad1.15x1.40mm_HandSolder, symbol Device:C
- added R?: 1M2, Resistor_SMD:R_0805_2012Metric_Pad1.15x1.40mm_HandSolder, symbol Device:R
- added R? (x3): 100k, Resistor_SMD:R_0805_2012Metric_Pad1.15x1.40mm_HandSolder, symbol Device:R
- added U?: L78L05_SOT89, Package_TO_SOT_SMD:SOT-89-3, symbol Regulator_Linear:L78L05_SOT89
- J?: value In1.2 -> In1.2 PolyMod
- R?: value 100k -> 200k
- R?: value 1k8 -> 1k82
- R?: value 360k -> 235k
- R?: value 5k6 -> 6k04
- R?: value 24k -> 26k7
- R?: value 1M5 -> 1M76
- RV?: value 10k -> 5k
Connections:
- net Vee is gone; now on net -5V: R?.2, RV?.1, RV?.2, U?.3 (VEE)
- net +12L: now also U?.3 (IN)
- net +12V: no longer C302.2
- net -12VA: now also R?.2
- net -5V: now also R?.2
- net GND: now also U?.3 (+), U?.7 (VHFT), C?.1, U?.2 (GND); no longer C306.1, C307.1, Q304.2 (E), R317.1, R320.2, R321.2
- net HardSyncIn3: no longer U?.6 (VHSI)
- net Inv1: no longer U?.2 (-)
- net Out1: no longer U?.1
- net PWM_In5: no longer R?.1
- net SoftSyncIn2: no longer U?.9 (VSSI)
- net poly: now reaches J?.T, R?.2
- net poly: now also R?.2
- net at R?.2, SW?.3 (C): no longer U?.3 (+)
- net at R?.1, U?.2 (SCALE2): now also R?.1
- new net: C?.2, U?.9 (VSSI)
- new net: R?.1, R?.2
- new net: R?.1, R?.1, R?.1, U?.2 (-)
- new net +5V: C302.2, U?.1 (OUT)
- new net GNDA: C306.1, C307.1, Q304.2 (E), R317.1, R320.2, R321.2
Other:
- moved on the sheet: C?, D?, J?, R?, RV?, U?A

Commit message: AS 3340 JE initiated
Parts:
- added C?: 10n, Capacitor_SMD:C_0805_2012Metric_Pad1.15x1.40mm_HandSolder, symbol Device:C
- added C?: 220p, Capacitor_SMD:C_0805_2012Metric_Pad1.15x1.40mm_HandSolder, symbol Device:C
- added C?: 100n, Capacitor_SMD:C_0805_2012Metric_Pad1.15x1.40mm_HandSolder, symbol Device:C
- added D?: Germanium, symbol Device:D
- added JP?: Jumper_3_Bridged12, Jumper:SolderJumper-3_P1.3mm_Bridged12_Pad1.0x1.5mm_NumberLabels, symbol Jumper:Jumper_3_Bridged12
- added Q?: MMBT3906, Package_TO_SOT_SMD:SOT-23, symbol Transistor_BJT:MMBT3906
- added R?: 100k, Resistor_SMD:R_0805_2012Metric_Pad1.15x1.40mm_HandSolder, symbol Device:R
- added R?: 10k, Resistor_SMD:R_0805_2012Metric_Pad1.15x1.40mm_HandSolder, symbol Device:R
- added R? (x2): OPEN, Resistor_SMD:R_0805_2012Metric_Pad1.15x1.40mm_HandSolder, symbol Device:R
- added R?: 20k, Resistor_SMD:R_0805_2012Metric_Pad1.15x1.40mm_HandSolder, symbol Device:R
- added R? (x2): 47k, Resistor_SMD:R_0805_2012Metric_Pad1.15x1.40mm_HandSolder, symbol Device:R
- C?: value 1n -> 1n alt
- C?: value 1n -> 1n poly; footprint Capacitor_SMD:C_0805_2012Metric_Pad1.15x1.40mm_HandSolder -> Capacitor_THT:C_Rect_L7.0mm_W2.0mm_P5.00mm
- RV?: footprint (none) -> Potentiometer_THT:Potentiometer_Bourns_3296W_Vertical
Connections:
- net +5V: now also JP?.1 (A)
- net -12VA: now also D?.2 (A)
- net GND: now also C?.2, D?.1 (K), D?.2 (A), C?.1, R?.1, R?.1, R?.1; no longer C?.1, D?.2 (A)
- net PWM_In5: now also D?.1 (K), U?.1, C?.2, R?.1
- net SoftSyncIn2: now also C?.2
- net VP_2: now also R?.2
- net VSO_3: now also Q?.2 (E), R?.2
- net VTO_1: now also R?.2
- net at C?.2, U?.11 (CAP): now also C?.1; no longer C?.2
- net at C?.2, U?.9 (VSSI): now also JP?.3 (B)
- net at D?.2 (A): now also R?.1, R?.1, R?.1, U?.2 (-), C?.1, R?.2
- new net: R?.1, R?.2
- new net: D?.1 (K), Q?.1 (B), R?.1, R?.1
- new net: C?.2, D?.2 (A), Q?.3 (C)
- new net: C?.1, R?.2
- new net: JP?.2 (C), R?.2
Other:
- note added: "1n timing cap\n0805 as backup\nTHT 1000 pf poly"
- note added: "Prophet 5"
- note added: "Prophet T8"
- moved on the sheet: C?, D?, J?, P?, R?, RV?, U?, U?A, U?C
