File: KicadJE_3340_RevA/KicadJE_AC3340_RevA _PCB.kicad_pcb (KiCad board)
At the start: 2 copper layers, 159 x 128 mm, 148 parts, among them J101 RampOut1, J102 PulseOut2, J103 SawOut3, J104 In1.1, J105 In1.2, J106 In1.3, J107 SS_In2, J108 HS_In3, J109 FM_In4, J110 PWM_In5, J111 SineOut4, P101 HEADER_2x5_Doepfer, Q101 MMBT3906, Q102 UMX1N, SW101 Octave (3 state), U101 TL072, U102 TL072, U103 TL072, U104 AS3340, U105 L78L05_SOT89, U106 L79L05_SOT89, U107 TL072

Commit message: Gerber
Parts:
- removed the G*** at (11.0, 161.0)
- removed H101, H102, H103, H104: MountingHole_Pad, AJ:MountingHole_Eurorack3
- removed H105: ON, AJ:LED_Hole_3mm
- removed TP101: Oct, AJ:Pot_6m3
- removed TP102: In1, AJ:Jack_6m3
- removed TP103: In2, AJ:Jack_6m3
- removed TP104: In3, AJ:Jack_6m3
- removed TP105: SS, AJ:Jack_6m3
- removed TP106: HS, AJ:Jack_6m3
- removed TP107: FM, AJ:Jack_6m3
- removed TP108: PWM, AJ:Jack_6m3
- removed TP109: Tri, AJ:Jack_6m3
- removed TP110: SQ, AJ:Jack_6m3
- removed TP111: Saw, AJ:Jack_6m3
- removed TP112: Fine, AJ:Pot_6m3_scale1
- removed TP113: PWM, AJ:Pot_6m3_scale1
- removed TP115: 3m5 jack, AJ:Jack_6m3
Other:
- board size 159 x 128 mm -> 40 x 100 mm
- board text removed: "AS3340 Rev A - 07/03-2020 Johansen Engineering"
- board text removed: "FM"
- board text removed: "Fine"
- board text removed: "HS"
- board text removed: "In 1"
- board text removed: "In 2"
- board text removed: "In 3"
- board text removed: "OCT"
- board text removed: "PWM"
- board text removed: "SQ"
- board text removed: "SS"
- board text removed: "Saw"
- board text removed: "Sine"
- board text removed: "Tri"
- board text removed: "in"
- board text removed: "out"
