File: KicadJE_3340_RevA/KicadJE_AC3340_RevA.sch (KiCad schematic (older format))
At the start: 147 parts, among them J101 RampOut1, J102 PulseOut2, J103 SawOut3, J104 In1.1, J105 In1.2, J106 In1.3, J107 SS_In2, J108 HS_In3, J109 FM_In4, J110 PWM_In5, J111 SineOut4, P101 HEADER_2x5_Doepfer, Q101 MMBT3906, Q102 UMX1N, SW101 Octave (3 state), U101 TL072, U102 TL072, U103 TL072, U104 AS3340, U105 L78L05_SOT89, U106 L79L05_SOT89, U107 TL072

Commit message: fix in sine section
Connections:
- net at Q102.6 (C), R140.1, R150.1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: no longer Q102.3 (C), R143.1, R149.1, U103.5 (+)
- new net: Q102.3 (C), R143.1, R149.1, U103.5 (+)
Changed lines of the file:
@@
 Wire Wire Line
 	5925 3475 5925 3525
-Wire Wire Line
-	5925 3475 6350 3475
 $Comp
 L Device:R R150
@@
 Wire Wire Line
 	6150 4700 6150 4675
-Connection ~ 6350 3475
-Wire Wire Line
-	6350 3475 6900 3475
 Text Notes 4550 3025 0    50   ~ 0
 Sine Shaper
@@
 	1    0    0    -1
 $EndComp
+Wire Wire Line
+	5925 3475 6900 3475
 $EndSCHEMATC

Commit message: Protection Diodes
Parts:
- removed D111: 1N1007, Diode_SMD:D_SOD-123, symbol Device:D
Changed lines of the file:
@@
 	2250 2700 2250 2875
 Connection ~ 2250 2875
-$Comp
-L Device:D D111
-U 1 1 5F4B950C
-P 2925 2650
-AR Path="/5F4B950C" Ref="D111"  Part="1"
-AR Path="/5D60ED9A/5F4B950C" Ref="D?"  Part="1"
-AR Path="/5CD6EBF4/5F4B950C" Ref="D?"  Part="1"
-AR Path="/5CE53731/5F4B950C" Ref="D?"  Part="1"
-AR Path="/5DD87D87/5F4B950C" Ref="D?"  Part="1"
-AR Path="/5F18E4B5/5F4B950C" Ref="D?"  Part="1"
-AR Path="/5E62ACA1/5F4B950C" Ref="D?"  Part="1"
-AR Path="/5E4B0DD9/5F4B950C" Ref="D?"  Part="1"
-AR Path="/5F49A670/5F4B950C" Ref="D?"  Part="1"
-F 0 "D111" H 2875 2750 50  0000 L CNN
-F 1 "1N1007" H 2750 2575 50  0000 L CNN
-F 2 "Diode_SMD:D_SOD-123" H 2925 2650 50  0001 C CNN
-F 3 "~" H 2925 2650 50  0001 C CNN
-	1    2925 2650
-	-1   0    0    1
-$EndComp
-Wire Wire Line
-	3075 2650 3425 2650
-Wire Wire Line
-	3425 2650 3425 2600
-Wire Wire Line
-	3425 2725 3425 2650
-Connection ~ 3425 2650
 Wire Wire Line
 	2950 2725 2975 2725
@@
 	2950 2725 2950 2875
 Wire Wire Line
-	2775 2875 2775 2650
-Wire Wire Line
 	2950 3075 2950 2875
 Wire Wire Line
@@
 Wire Wire Line
 	2575 2700 2600 2700
-Wire Wire Line
-	2250 2875 2775 2875
 Connection ~ 2875 2875
 Wire Wire Line
 	2875 2875 2950 2875
 Connection ~ 2950 2875
-Connection ~ 2775 2875
-Wire Wire Line
-	2775 2875 2875 2875
 Wire Wire Line
 	2950 2875 3400 2875
@@
 Wire Wire Line
 	5925 3475 6900 3475
+Wire Wire Line
+	3425 2600 3425 2725
+Wire Wire Line
+	2250 2875 2875 2875
 $EndSCHEMATC

Commit message: Saved in newer kicad
Parts:
- RV101, RV102: symbol Envelope-cache-2018-08-04-13-00-04:POT -> KicadJE_AC3340_RevA-rescue:POT-Envelope-cache-2018-08-04-13-00-04
Changed lines of the file:
@@
 EESchema Schematic File Version 4
-EELAYER 29 0
+EELAYER 30 0
 EELAYER END
 $Descr A4 11693 8268
@@
 	1175 4525 1425 4525
 $Comp
-L Envelope-cache-2018-08-04-13-00-04:GND #PWR0103
+L KicadJE_AC3340_RevA-rescue:GND-Envelope-cache-2018-08-04-13-00-04 #PWR0103
 U 1 1 5F4B92B1
 P 1325 6275
@@
 	1200 2875 1450 2875
 $Comp
-L Envelope-cache-2018-08-04-13-00-04:GND #PWR0104
+L KicadJE_AC3340_RevA-rescue:GND-Envelope-cache-2018-08-04-13-00-04 #PWR0104
 U 1 1 5F4B93A7
 P 1350 3425
@@
 $EndComp
 $Comp
-L Envelope-cache-2018-08-04-13-00-04:POT RV?
+L KicadJE_AC3340_RevA-rescue:POT-Envelope-cache-2018-08-04-13-00-04 RV?
 U 1 1 5F4B9436
 P 2800 7125
@@
 Connection ~ 2250 2475
 $Comp
-L Envelope-cache-2018-08-04-13-00-04:GND #PWR0109
+L KicadJE_AC3340_RevA-rescue:GND-Envelope-cache-2018-08-04-13-00-04 #PWR0109
 U 1 1 5F4B952E
 P 2250 2575
@@
 Connection ~ 2600 2025
 $Comp
-L Envelope-cache-2018-08-04-13-00-04:GND #PWR0108
+L KicadJE_AC3340_RevA-rescue:GND-Envelope-cache-2018-08-04-13-00-04 #PWR0108
 U 1 1 5F4B9562
 P 2250 2150
@@
 	3275 2725 3425 2725
 $Comp
-L Envelope-cache-2018-08-04-13-00-04:GND #PWR0112
+L KicadJE_AC3340_RevA-rescue:GND-Envelope-cache-2018-08-04-13-00-04 #PWR0112
 U 1 1 5F4B9576
 P 2325 1425
@@
 $EndComp
 $Comp
-L Envelope-cache-2018-08-04-13-00-04:GND #PWR0134
+L KicadJE_AC3340_RevA-rescue:GND-Envelope-cache-2018-08-04-13-00-04 #PWR0134
 U 1 1 5F4F8A5B
 P 6225 5675
@@
 $EndComp
 $Comp
-L Envelope-cache-2018-08-04-13-00-04:GND #PWR0128
+L KicadJE_AC3340_RevA-rescue:GND-Envelope-cache-2018-08-04-13-00-04 #PWR0128
 U 1 1 5F4F8A76
 P 5575 5675
@@
 	8175 5325 8175 5275
 $Comp
-L Envelope-cache-2018-08-04-13-00-04:+5V #PWR?
+L KicadJE_AC3340_RevA-rescue:+5V-Envelope-cache-2018-08-04-13-00-04 #PWR?
 U 1 1 5F4F8AF5
 P 8175 5225
@@
 Connection ~ 2925 3475
 $Comp
-L Envelope-cache-2018-08-04-13-00-04:GND #PWR0118
+L KicadJE_AC3340_RevA-rescue:GND-Envelope-cache-2018-08-04-13-00-04 #PWR0118
 U 1 1 5F56AA41
 P 3350 3900
@@
 	6475 2600 6275 2600
 $Comp
-L Envelope-cache-2018-08-04-13-00-04:GND #PWR0137
+L KicadJE_AC3340_RevA-rescue:GND-Envelope-cache-2018-08-04-13-00-04 #PWR0137
 U 1 1 5F66CD58
 P 6725 2600
@@
 Connection ~ 5275 1900
 $Comp
-L Envelope-cache-2018-08-04-13-00-04:+5V #PWR?
+L KicadJE_AC3340_RevA-rescue:+5V-Envelope-cache-2018-08-04-13-00-04 #PWR?
 U 1 1 5F66CDDA
 P 5025 1350
@@
 $EndComp
 $Comp
-L Envelope-cache-2018-08-04-13-00-04:+5V #PWR?
+L KicadJE_AC3340_RevA-rescue:+5V-Envelope-cache-2018-08-04-13-00-04 #PWR?
 U 1 1 5F6F74CC
 P 850 6750
@@
 $EndComp
 $Comp
-L Envelope-cache-2018-08-04-13-00-04:GND #PWR0102
+L KicadJE_AC3340_RevA-rescue:GND-Envelope-cache-2018-08-04-13-00-04 #PWR0102
 U 1 1 5F6F8CBF
 P 850 7500
@@
 Connection ~ 2925 4850
 $Comp
-L Envelope-cache-2018-08-04-13-00-04:GND #PWR0121
+L KicadJE_AC3340_RevA-rescue:GND-Envelope-cache-2018-08-04-13-00-04 #PWR0121
 U 1 1 5FE418BD
 P 3450 4925
@@
 Connection ~ 2925 5650
 $Comp
-L Envelope-cache-2018-08-04-13-00-04:GND #PWR0122
+L KicadJE_AC3340_RevA-rescue:GND-Envelope-cache-2018-08-04-13-00-04 #PWR0122
 U 1 1 5FE7E315
 P 3450 5725
@@
 Connection ~ 8250 1350
 $Comp
-L Envelope-cache-2018-08-04-13-00-04:GND #PWR0144
+L KicadJE_AC3340_RevA-rescue:GND-Envelope-cache-2018-08-04-13-00-04 #PWR0144
 U 1 1 6047E7D0
 P 8625 1350
@@
 $EndComp
 $Comp
-L Envelope-cache-2018-08-04-13-00-04:GND #PWR0145
+L KicadJE_AC3340_RevA-rescue:GND-Envelope-cache-2018-08-04-13-00-04 #PWR0145
 U 1 1 605CBE50
 P 8950 2425
@@
 	5575 3725 5475 3725
 $Comp
-L Envelope-cache-2018-08-04-13-00-04:GND #PWR0127
+L KicadJE_AC3340_RevA-rescue:GND-Envelope-cache-2018-08-04-13-00-04 #PWR0127
 U 1 1 608519AE
 P 5575 4100
@@
 $EndComp
 $Comp
-L Envelope-cache-2018-08-04-13-00-04:GND #PWR0136
+L KicadJE_AC3340_RevA-rescue:GND-Envelope-cache-2018-08-04-13-00-04 #PWR0136
 U 1 1 6091DDBA
 P 6675 4100
@@
 	9000 2425 8950 2425
 $Comp
-L Envelope-cache-2018-08-04-13-00-04:GND #PWR0124
+L KicadJE_AC3340_RevA-rescue:GND-Envelope-cache-2018-08-04-13-00-04 #PWR0124
 U 1 1 60D96B00
 P 4100 7325
@@
 	3900 7125 3950 7125
 $Comp
-L Envelope-cache-2018-08-04-13-00-04:POT RV?
+L KicadJE_AC3340_RevA-rescue:POT-Envelope-cache-2018-08-04-13-00-04 RV?
 U 1 1 60D4C6A7
 P 4100 7125
@@
 	6025 6825 5850 6825
 $Comp
-L Envelope-cache-2018-08-04-13-00-04:GND #PWR0125
+L KicadJE_AC3340_RevA-rescue:GND-Envelope-cache-2018-08-04-13-00-04 #PWR0125
 U 1 1 615A670C
 P 7625 4550
@@
 $EndComp
 $Comp
-L Envelope-cache-2018-08-04-13-00-04:GND #PWR0142
+L KicadJE_AC3340_RevA-rescue:GND-Envelope-cache-2018-08-04-13-00-04 #PWR0142
 U 1 1 5E789A07
 P 4925 7400
@@
 Connection ~ 6925 6350
 $Comp
-L Envelope-cache-2018-08-04-13-00-04:GND #PWR0120
+L KicadJE_AC3340_RevA-rescue:GND-Envelope-cache-2018-08-04-13-00-04 #PWR0120
 U 1 1 5EF57B05
 P 6800 6350
@@
 	6800 6350 6925 6350
 $Comp
-L Envelope-cache-2018-08-04-13-00-04:GND #PWR0147
+L KicadJE_AC3340_RevA-rescue:GND-Envelope-cache-2018-08-04-13-00-04 #PWR0147
 U 1 1 5EF95D3D
 P 4275 7175
@@
 $EndComp
 $Comp
-L Envelope-cache-2018-08-04-13-00-04:GND #PWR0146
+L KicadJE_AC3340_RevA-rescue:GND-Envelope-cache-2018-08-04-13-00-04 #PWR0146
 U 1 1 5EF966DD
 P 2250 7375
