File: KicadJE_3340_RevB/KicadJE_AC3340_RevB.kicad_pcb (KiCad board)
At the start: 2 copper layers, 159 x 128 mm, 148 parts, among them J101 RampOut1, J102 PulseOut2, J103 SawOut3, J104 In1.1, J105 In1.2, J106 In1.3, J107 SS_In2, J108 HS_In3, J109 FM_In4, J110 PWM_In5, J111 SineOut4, P101 HEADER_2x5_Doepfer, Q101 MMBT3906, Q102 UMX1N, SW101 Octave (3 state), U101 TL072, U102 TL072, U103 TL072, U104 AS3340, U105 L78L05_SOT89, U106 L79L05_SOT89, U107 TL072

Commit message: long time ago
Other:
- net class Default removed
- net class Power removed
